Commit message: working in gazebo sim with some problems

File: model/robot.xacro (robot description, xacro)
@@ -32,116 +32,202 @@
     <!-- Body Link -->
     <link name="body_link">
-        <visual>
-            <origin xyz="0.0 0.0 0.0" rpy="0.0 0.0 0.0"/>
-            <geometry>
-                <box size="${body_length} ${body_width} ${body_height}"/>
-            </geometry>
-            <material name="body_material">
-                <color rgba="0.25 0.25 0.25 1.0"/>
-            </material>
-        </visual>
-        <collision>
-            <origin xyz="0.0 0.0 0.0" rpy="0.0 0.0 0.0"/>
-            <geometry>
-                <box size="${body_length} ${body_width} ${body_height}"/>
-            </geometry>
-        </collision>
-        <inertial>
-            <mass value="10"/>
-            <inertia ixx="${body_inertia_x}" ixy="0.0" ixz="0.0" iyy="${body_inertia_y}" iyz="0" izz="${body_inertia_z}"/>
-            <origin xyz="0 0 0" rpy="0 0 0"/>
-        </inertial>
+        <inertial>
+        <origin
+            xyz="-0.0283919190232791 2.73258068193935E-08 -0.00802366185586431"
+            rpy="0 0 0" />
+        <mass
+            value="0.147758674199692" />
+        <inertia
+            ixx="0.000290930982603083"
+            ixy="2.96592562996834E-10"
+            ixz="-4.89953593135407E-06"
+            iyy="0.000293366944607641"
+            iyz="-1.24079970534305E-11"
+            izz="0.000578469246893076" />
+        </inertial>
+        <visual>
+        <origin
+            xyz="0 0 0"
+            rpy="0 0 0" />
+        <geometry>
+            <mesh
+            filename="package://gazebo_differential_drive_robot/meshes/base_link.STL" />
+        </geometry>
+        <material
+            name="">
+            <color
+            rgba="0.792156862745098 0.819607843137255 0.933333333333333 1" />
+        </material>
+        </visual>
+        <collision>
+        <origin
+            xyz="0 0 0"
+            rpy="0 0 0" />
+        <geometry>
+            <mesh
+            filename="package://gazebo_differential_drive_robot/meshes/base_link.STL" />
+        </geometry>
+        </collision>
     </link>
     <!-- Left Wheel -->
     <link name="left_wheel_link">
-        <visual>
-            <origin xyz="0.0 0.0 0.0" rpy="1.570795 0.0 0.0"/>
-            <geometry>
-                <cylinder radius="${wheel_radius}" length="${wheel_width}"/>
-            </geometry>
-            <material name="wheel_material">
-                <color rgba="0.0 0.0 0.0 1.0"/>
-            </material>
-        </visual>
-        <collision>
-            <origin xyz="0.0 0.0 0.0" rpy="1.570795 0.0 0.0"/>
-            <geometry>
-                <cylinder radius="${wheel_radius}" length="${wheel_width}"/>
-            </geometry>
-        </collision>
-        <inertial>
-            <mass value="2"/>
-            <inertia ixx="${wheel_inertia_x}" ixy="0.0" ixz="0.0" iyy="${wheel_inertia_y}" iyz="0" izz="${wheel_inertia_z}"/>
-            <origin xyz="0.0 0.0 0.0" rpy="1.570795 0.0 0.0"/>
-        </inertial>
+        <inertial>
+        <origin
+            xyz="2.35316488517157E-11 -1.95061293506438E-11 0.00807930941679115"
+            rpy="0 0 0" />
+        <mass
+            value="0.00843740400988768" />
+        <inertia
+            ixx="1.23422492282635E-06"
+            ixy="-1.48859597124639E-10"
+            ixz="3.30647721519471E-16"
+            iyy="1.23431714543936E-06"
+            iyz="-6.17403432705978E-16"
+            izz="2.19640206701058E-06" />
+        </inertial>
+        <visual>
+        <origin
+            xyz="0 0 0"
+            rpy="0 0 0" />
+        <geometry>
+            <mesh
+            filename="package://gazebo_differential_drive_robot/meshes/left_wheel_link.STL" />
+        </geometry>
+        <material
+            name="">
+            <color
+            rgba="0.792156862745098 0.819607843137255 0.933333333333333 1" />
+        </material>
+        </visual>
+        <collision>
+        <origin
+            xyz="0 0 0"
+            rpy="0 0 0" />
+        <geometry>
+            <mesh
+            filename="package://gazebo_differential_drive_robot/meshes/left_wheel_link.STL" />
+        </geometry>
+        </collision>
     </link>
     <!-- Right Wheel -->
     <link name="right_wheel_link">
-        <visual>
-            <origin xyz="0.0 0.0 0.0" rpy="1.570795 0.0 0.0"/>
-            <geometry>
-                <cylinder radius="${wheel_radius}" length="${wheel_width}"/>
-            </geometry>
-            <material name="wheel_material">
-                <color rgba="0.0 0.0 0.0 1.0"/>
-            </material>
-        </visual>
-        <collision>
-            <origin xyz="0.0 0.0 0.0" rpy="1.570795 0.0 0.0"/>
-            <geometry>
-                <cylinder radius="${wheel_radius}" length="${wheel_width}"/>
-            </geometry>
-        </collision>
-        <inertial>
-            <mass value="2"/>
-            <inertia ixx="${wheel_inertia_x}" ixy="0.0" ixz="0.0" iyy="${wheel_inertia_y}" iyz="0" izz="${wheel_inertia_z}"/>
-            <origin xyz="0.0 0.0 0.0" rpy="1.570795 0.0 0.0"/>
-        </inertial>
+        <inertial>
+        <origin
+            xyz="1.16513049208677E-11 2.82576566312809E-11 0.00807967326089072"
+            rpy="0 0 0" />
+        <mass
+            value="0.00843740400988766" />
+        <inertia
+            ixx="1.23422492920575E-06"
+            ixy="1.48861577857816E-10"
+            ixz="4.91594534149496E-16"
+            iyy="1.23431713905996E-06"
+            iyz="4.98850564443408E-16"
+            izz="2.19640206701057E-06" />
+        </inertial>
+        <visual>
+        <origin
+            xyz="0 0 0"
+            rpy="0 0 0" />
+        <geometry>
+            <mesh
+            filename="package://gazebo_differential_drive_robot/meshes/right_wheel_link.STL" />
+        </geometry>
+        <material
+            name="">
+            <color
+            rgba="0.792156862745098 0.819607843137255 0.933333333333333 1" />
+        </material>
+        </visual>
+        <collision>
+        <origin
+            xyz="0 0 0"
+            rpy="0 0 0" />
+        <geometry>
+            <mesh
+            filename="package://gazebo_differential_drive_robot/meshes/right_wheel_link.STL" />
+        </geometry>
+        </collision>
     </link>
     <!-- Caster Wheel -->
     <link name="caster_link">
-        <visual>
-            <origin xyz="0.0 0.0 0.0" rpy="0.0 0.0 0.0"/>
+        <inertial>
+            <origin
+                xyz="1.38777878078145E-17 3.46944695195361E-18 -2.40838632757448E-20"
+                rpy="0 0 0" />
+            <mass
+                value="0.0669259238391975" />
+            <inertia
+                ixx="4.31779290240967E-06"
+                ixy="3.54080995565633E-23"
+                ixz="-7.16933357795495E-22"
+                iyy="4.31779290240967E-06"
+                iyz="6.61721086913841E-23"
+                izz="4.31779290240967E-06" />
+        </inertial>
+        <visual>
+            <origin
+                xyz="0 0 0"
+                rpy="0 0 0" />
             <geometry>
-                <sphere radius="${caster_radius}"/>
+                <mesh
+                filename="package://gazebo_differential_drive_robot/meshes/castor_wheel_xz_link.STL" />
             </geometry>
-            <material name="caster_material">
-                <color rgba="0.0 0.0 0.0 1.0"/>
+            <material
+                name="">
+                <color
+                rgba="1 1 1 1" />
             </material>
         </visual>
         <collision>
-            <origin xyz="0.0 0.0 0.0" rpy="0.0 0.0 0.0"/>
+            <origin
+                xyz="0 0 0"
+                rpy="0 0 0" />
             <geometry>
-                <sphere radius="${caster_radius}"/>
+                <mesh
+                filename="package://gazebo_differential_drive_robot/meshes/castor_wheel_xz_link.STL" />
             </geometry>
         </collision>
-        <inertial>
-            <mass value="0.5"/>
-            <inertia ixx="${caster_inertia_x}" ixy="0.0" ixz="0.0" iyy="${caster_inertia_y}" iyz="0" izz="${caster_inertia_z}"/>
-            <origin xyz="0 0 0" rpy="0 0 0"/>
-        </inertial>
     </link>
     <!-- Joints -->
     <!-- Left Wheel Joint -->
     <joint name="left_wheel_joint" type="continuous">
-        <origin xyz="-${wheel_offset} ${wheel_separation/2} -${wheel_radius/2}" rpy="0 0 0"/>
-        <parent link="body_link"/>
-        <child link="left_wheel_link"/>
-        <axis xyz="0 1 0"/>
-        <limit effort="100" velocity="10.0"/>
-        <dynamics damping="0.1" friction="0.1"/>
+        <origin
+            xyz="-0.0775 0.0857 -0.0180000000000005"
+            rpy="-1.5707963267949 0 0" />
+        <parent
+            link="body_link" />
+        <child
+            link="left_wheel_link" />
+        <axis
+            xyz="0 0 1" />
+        <limit
+            effort="3"
+            velocity="5" />
+        <dynamics
+            friction="0.1" />
     </joint>
     <!-- Right Wheel Joint -->
     <joint name="right_wheel_joint" type="continuous">
-        <origin xyz="-${wheel_offset} ${-wheel_separation/2} -${wheel_radius/2}" rpy="0 0 0"/>
-        <parent link="body_link"/>
-        <child link="right_wheel_link"/>
-        <axis xyz="0 1 0"/>
-        <limit effort="100" velocity="10.0"/>
-        <dynamics damping="0.1" friction="0.1"/>
+        <origin
+            xyz="-0.0775 -0.0857 -0.0180000000000005"
+            rpy="-1.5707963267949 0 -3.1415926535898" />
+        <parent
+            link="body_link" />
+        <child
+            link="right_wheel_link" />
+        <axis
+            xyz="0 0 -1" />
+        <limit
+            effort="3"
+            velocity="5" />
+        <dynamics
+            friction="0.1" />
     </joint>
     <!-- Caster Wheel Joint (fixed) -->
     <joint name="caster_joint" type="fixed">
-        <origin xyz="${caster_offset} 0 -${caster_radius/2}" rpy="0 0 0"/>
+        <origin
+            xyz="0 0 0"
+            rpy="1.5707963267949 0 0" />
         <parent link="body_link"/>
         <child link="caster_link"/>

Commit message: fixed urdf

File: model/robot.xacro (robot description, xacro)
@@ -3,7 +3,7 @@
     <!-- Robot Parameters -->
     <xacro:property name="PI" value="3.14159265"/>
-    <xacro:property name="body_length" value="0.5"/>
-    <xacro:property name="body_width" value="0.3"/>
-    <xacro:property name="body_height" value="0.1"/>
+    <xacro:property name="body_length" value="0.18"/>
+    <xacro:property name="body_width" value="0.17"/>
+    <xacro:property name="body_height" value="0.01"/>
     <xacro:property name="body_density" value="7850.0"/> <!-- Steel -->
     <xacro:property name="body_mass" value="${body_density * body_length * body_height * body_width}"/>
@@ -11,6 +11,6 @@
     <xacro:property name="body_inertia_y" value="${1.0/12.0 * body_mass * (body_length*body_length + body_height*body_height)}"/>
     <xacro:property name="body_inertia_z" value="${1.0/12.0 * body_mass * (body_length*body_length + body_width*body_width)}"/>
-    <xacro:property name="wheel_radius" value="0.1"/>
-    <xacro:property name="wheel_width" value="0.05"/>
+    <xacro:property name="wheel_radius" value="0.04"/>
+    <xacro:property name="wheel_width" value="0.015"/>
     <xacro:property name="wheel_separation" value="${body_width + wheel_width}"/>
     <xacro:property name="wheel_offset" value="${body_length/2 - wheel_radius}"/>
@@ -20,5 +20,5 @@
     <xacro:property name="wheel_inertia_y" value="${1.0/12.0 * wheel_mass * (3*wheel_radius*wheel_radius + wheel_width*wheel_width)}"/>
     <xacro:property name="wheel_inertia_z" value="${1.0/2.0 * wheel_mass * wheel_radius * wheel_radius}"/>
-    <xacro:property name="caster_radius" value="0.1"/>
+    <xacro:property name="caster_radius" value="0.0125"/>
     <xacro:property name="caster_offset" value="${body_length/2 - caster_radius}"/>
     <xacro:property name="caster_density" value="0.1"/>
@@ -34,8 +34,8 @@
         <inertial>
         <origin
-            xyz="-0.0283919190232791 2.73258068193935E-08 -0.00802366185586431"
+            xyz="-0.0284 0 -0.008"
             rpy="0 0 0" />
         <mass
-            value="0.147758674199692" />
+            value="0.300" />
         <inertia
             ixx="0.000290930982603083"
@@ -47,25 +47,24 @@
         </inertial>
         <visual>
-        <origin
-            xyz="0 0 0"
-            rpy="0 0 0" />
-        <geometry>
-            <mesh
-            filename="package://gazebo_differential_drive_robot/meshes/base_link.STL" />
-        </geometry>
-        <material
-            name="">
-            <color
-            rgba="0.792156862745098 0.819607843137255 0.933333333333333 1" />
-        </material>
-        </visual>
-        <collision>
-        <origin
-            xyz="0 0 0"
-            rpy="0 0 0" />
-        <geometry>
-            <mesh
-            filename="package://gazebo_differential_drive_robot/meshes/base_link.STL" />
-        </geometry>
+            <origin
+                xyz="0 0 0"
+                rpy="0 0 0" />
+            <geometry>
+                <mesh
+                filename="package://gazebo_differential_drive_robot/meshes/base_link.STL" />
+            </geometry>
+            <material
+                name="">
+                <color
+                rgba="0.792156862745098 0.819607843137255 0.933333333333333 1" />
+            </material>
+        </visual>
+        <collision>
+            <origin
+                xyz="0 0 0"
+                rpy="0 0 0" />
+            <geometry>
+                <box size="0.18 0.17 0.03" />
+            </geometry>
         </collision>
     </link>
@@ -74,8 +73,8 @@
         <inertial>
         <origin
-            xyz="2.35316488517157E-11 -1.95061293506438E-11 0.00807930941679115"
+            xyz="0 0 0.00808"
             rpy="0 0 0" />
         <mass
-            value="0.00843740400988768" />
+            value="0.015" />
         <inertia
             ixx="1.23422492282635E-06"
@@ -101,11 +100,10 @@
         </visual>
         <collision>
-        <origin
-            xyz="0 0 0"
-            rpy="0 0 0" />
-        <geometry>
-            <mesh
-            filename="package://gazebo_differential_drive_robot/meshes/left_wheel_link.STL" />
-        </geometry>
+            <origin
+                xyz="0 0 0"
+                rpy="0 0 0" />
+            <geometry>
+                <cylinder radius="0.02" length="0.015"/>
+            </geometry>
         </collision>
     </link>
@@ -114,8 +112,8 @@
         <inertial>
         <origin
-            xyz="1.16513049208677E-11 2.82576566312809E-11 0.00807967326089072"
+            xyz="0 0 0.00808"
             rpy="0 0 0" />
         <mass
-            value="0.00843740400988766" />
+            value="0.015" />
         <inertia
             ixx="1.23422492920575E-06"
@@ -145,6 +143,5 @@
             rpy="0 0 0" />
         <geometry>
-            <mesh
-            filename="package://gazebo_differential_drive_robot/meshes/right_wheel_link.STL" />
+            <cylinder radius="0.02" length="0.015"/>
         </geometry>
         </collision>
@@ -154,6 +151,6 @@
         <inertial>
             <origin
-                xyz="1.38777878078145E-17 3.46944695195361E-18 -2.40838632757448E-20"
-                rpy="0 0 0" />
+                xyz="0.0 0 0.0"
+                rpy="-1.5707963267949 0 0" />
             <mass
                 value="0.0669259238391975" />
@@ -182,9 +179,8 @@
         <collision>
             <origin
-                xyz="0 0 0"
-                rpy="0 0 0" />
-            <geometry>
-                <mesh
-                filename="package://gazebo_differential_drive_robot/meshes/castor_wheel_xz_link.STL" />
+                xyz="0.0 0 -0.0"
+                rpy="0 0 0" />
+            <geometry>
+                <sphere radius=".0125" />
             </geometry>
         </collision>
@@ -194,5 +190,5 @@
     <joint name="left_wheel_joint" type="continuous">
         <origin
-            xyz="-0.0775 0.0857 -0.0180000000000005"
+            xyz="-0.0775 0.0925 -0.02"
             rpy="-1.5707963267949 0 0" />
         <parent
@@ -211,5 +207,5 @@
     <joint name="right_wheel_joint" type="continuous">
         <origin
-            xyz="-0.0775 -0.0857 -0.0180000000000005"
+            xyz="-0.0775 -0.0925 -0.02"
             rpy="-1.5707963267949 0 -3.1415926535898" />
         <parent
@@ -228,6 +224,6 @@
     <joint name="caster_joint" type="fixed">
         <origin
-            xyz="0 0 0"
-            rpy="1.5707963267949 0 0" />
+            xyz="0.07075 0 -0.0125"
+            rpy="-1.5707963267949 0 0" />
         <parent link="body_link"/>
         <child link="caster_link"/>
